Commit message: now atlas has a model

File: atlas_perception_description/urdf/car_macro.urdf.xacro (robot description, xacro)
@@ -5,7 +5,7 @@
         <link name="${prefix}base_link">
             <visual>
-                <origin xyz="0 0 0" rpy="0 0 0" />
+                <origin xyz="-0.9 0 -0.5" rpy="0 0 0" />
                 <geometry>
-                    <mesh filename="package://atlas_perception_description/meshes/mitsubishi_miev.stl" />
+                    <mesh filename="package://atlas_perception_description/meshes/mitsubishi_miev.dae" />
                 </geometry>
             </visual>
