Commit message: aruco detect is now implemented

File: atlas_perception_description/urdf/atlas_macro.urdf.xacro (robot description, xacro)
@@ -3,4 +3,6 @@
     xmlns:xacro="http://www.ros.org/wiki/xacro">
     <xacro:include filename="$(find atlas_perception_description)/urdf/car_macro.urdf.xacro" />
+    <xacro:include filename="$(find pointgrey_camera_description)/urdf/pointgrey_flea3.urdf.xacro" />
+    <xacro:include filename="$(find lms1xx)/urdf/sick_lms1xx.urdf.xacro" />
     <xacro:macro name="atlas" params="prefix">
         <link name="${prefix}base_link" />
@@ -11,4 +13,22 @@
             <child link="${prefix}car_base_link" />
         </joint>
+        <xacro:pointgrey_flea3 frame="${prefix}frontal_camera" />
+        <joint name="${prefix}base_link_to_${prefix}frontal_camera" type="fixed">
+            <origin xyz="0 -0.1 0.2" rpy="0 0 ${-pi/2}" />
+            <parent link="${prefix}base_link" />
+            <child link="${prefix}frontal_camera" />
+        </joint>
+        <xacro:sick_lms1xx frame="${prefix}frontal_laser_left" />
+        <joint name="${prefix}base_link_to_${prefix}frontal_laser_left" type="fixed">
+            <origin xyz="0.6 0 0" rpy="0 0 ${-pi/3}" />
+            <parent link="${prefix}base_link" />
+            <child link="${prefix}frontal_laser_left" />
+        </joint>
+        <xacro:sick_lms1xx frame="${prefix}frontal_laser_right" />
+        <joint name="${prefix}base_link_to_${prefix}frontal_laser_right" type="fixed">
+            <origin xyz="-0.6 0 0" rpy="0 0 ${-2*pi/3}" />
+            <parent link="${prefix}base_link" />
+            <child link="${prefix}frontal_laser_right" />
+        </joint>
     </xacro:macro>
 </robot>

Commit message: tablier marker is working

File: atlas_perception_description/urdf/atlas_macro.urdf.xacro (robot description, xacro)
@@ -31,4 +31,10 @@
             <child link="${prefix}frontal_laser_right" />
         </joint>
+        <link name="${prefix}tablier_marker" />
+        <joint name="${prefix}frontal_camera_optical_to_${prefix}tablier_marker" type="fixed">
+            <origin xyz="-0.0515 -0.1984 -0.8176" rpy="${pi+0.5} -0.2 ${-pi/2}" />
+            <parent link="${prefix}frontal_camera_optical" />
+            <child link="${prefix}tablier_marker" />
+        </joint>
     </xacro:macro>
 </robot>
